File: PS-PowerSelectorPCB.kicad_pcb (KiCad board)
At the start: 2 copper layers, 47.6 x 44.2 mm, 27 parts, among them J1 SuppChargerIn, J2 PowerSupplyIn, J3 SuppChargerOut, J4 PowerSupplyOut, J5 Signals, J6 HV_Lockout

Commit message: fixed switch footprint + silkscreen
Parts:
- removed S1: 100DP1T2B4VS2QE, footprints:100DP1T2B4VS2QE
- added SW1: Power Source Selector, footprints:100DP1T2B4VS2QE, F.Cu at (91.2, 114.6)
Other:
- board text added: "SUPP BATTERY"
- board text removed: "SUPP CHARGER"
