File: PS-PowerSelectorPCB.kicad_pcb (KiCad board)
At the start: 2 copper layers, 47.6 x 44.2 mm, 27 parts, among them J1 SuppChargerIn, J2 PowerSupplyIn, J3 SuppChargerOut, J4 PowerSupplyOut, J5 Signals, J6 HV_Lockout, SW1 Power Source Selector

Commit message: silkscreens
Parts:
- added G***: LOGO, LOGO, F.Cu at (106.0, 98.8)
- added G***: LOGO, LOGO, F.Cu at (85.5, 99.1)
- added G***: LOGO, LOGO, B.Cu at (78.0, 92.6)
- added G***: LOGO, LOGO, B.Cu at (86.4, 108.9)
- J6: moved to F.Cu
- moved H3 1.68 mm to (115.8, 86.2)
- moved J6 1.67 mm to (78.3, 99.5)
- moved LOGO1 1.63 mm to (105.8, 125.2)
- moved H2 1.35 mm to (116.2, 123.5)
- moved J1 1.24 mm to (85.1, 90.0)
- moved J4 1.22 mm to (113.3, 93.6)
- moved J5 0.70 mm to (78.4, 117.5)
- moved H4 0.63 mm to (77.4, 123.6)
- moved H1 0.53 mm to (77.4, 86.2)
- moved J2 0.45 mm to (102.0, 87.8)
- moved J3 0.34 mm to (112.6, 108.1)
Routing:
- net PS+: track 17.4 -> 24.6 mm
- net /HV_LO-: track 11.2 -> 14.4 mm
- net /HV_LO+: track 16.7 -> 14.3 mm
- net SuppChargerIn+: track 17.3 -> 18.5 mm
- net /LED+: track 23.5 -> 23.0 mm
Other:
- board size 47.6 x 44.2 mm -> 45.8 x 44.3 mm
- board text added: "AHHHH"

Commit message: gerbers + fixes
Parts:
- removed the G*** at (86.4, 108.9)
- F1: moved to F.Cu
- J5, J6: moved to B.Cu
- moved J5 12.6 mm to (78.3, 105.0)
- moved F2 11.8 mm to (82.3, 105.5), turned to 90 degrees
- moved J6 2.68 mm to (78.1, 96.8)
- moved J4 2.62 mm to (115.9, 93.6)
- moved J3 1.88 mm to (114.5, 108.1)
- moved G*** 1.79 mm to (83.7, 99.1)
- moved G*** 1.46 mm to (107.4, 99.1)
- moved LOGO2 0.88 mm to (100.5, 108.1)
Routing:
- net PS+: track 24.6 -> 29.2 mm
- net /LV_EN_PS: track 31.9 -> 35.9 mm
- net SuppChargerOut+: track 15.3 -> 16.8 mm
- net /LV_EN_FUSED: track 24.9 -> 24.0 mm
- net /LV_EN_SUPP: track 22.0 -> 21.0 mm
- net /LV_EN_IN: track 4.87 -> 4.24 mm

Commit message: filled zones
Parts:
- removed the G*** at (83.7, 99.1)
- D6, D7, G***: moved to F.Cu
- moved G*** 32.3 mm to (110.1, 95.8), turned to 0 degrees
- moved G*** 24.3 mm to (83.1, 99.2)
- moved D6 3.81 mm to (106.3, 99.2), turned to 180 degrees
- moved D7 1.32 mm to (106.3, 101.7), turned to 180 degrees
Routing:
- net PS+: track 29.2 -> 0.00 mm
- net LV-: track 4.25 -> 6.56 mm, vias 2 -> 0
- net /SC_Fused: track 29.9 -> 27.9 mm
- net /LED+: track 23.0 -> 22.9 mm, vias 1 -> 0
- added copper zone on F.Cu, net LV-
- added copper zone on F.Cu, net PS+

Commit message: added step
Routing:
- net /LV_EN_FUSED: vias 1 -> 0
- net /LV_EN_SUPP: vias 1 -> 0
Changed lines of the file:
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@@
 		)
 		(property "Value" "Signals"
-			(at 3.27 -6.35 -90)
+			(at 3.27 -6.35 270)
 			(layer "B.SilkS" knockout)
 			(effects
@@
 		)
 		(property "Value" "HV_Lockout"
-			(at 3.125 -1 -90)
+			(at 3.125 -1 270)
 			(layer "B.SilkS" knockout)
 			(effects
@@
 	)
 	(segment
+		(start 95.875 111.575)
+		(end 95.875 114.57)
+		(width 0.5)
+		(layer "F.Cu")
+		(net 11)
+	)
+	(segment
 		(start 95.9 108.575)
 		(end 96.775 107.7)
@@
 		(net 11)
 	)
-	(via
-		(at 95.9 111.55)
-		(size 0.6)
-		(drill 0.3)
-		(layers "F.Cu" "B.Cu")
+	(segment
+		(start 95.9 111.55)
+		(end 95.875 111.575)
+		(width 0.5)
+		(layer "F.Cu")
 		(net 11)
 	)
@@
 	)
 	(segment
-		(start 95.9 114.57)
-		(end 95.9 111.55)
-		(width 0.5)
-		(layer "B.Cu")
-		(net 11)
-	)
-	(segment
 		(start 108.1375 107.625)
 		(end 114.025 107.625)
@@
 	)
 	(segment
+		(start 91.175 111.575)
+		(end 91.175 114.57)
+		(width 0.5)
+		(layer "F.Cu")
+		(net 17)
+	)
+	(segment
 		(start 91.2 108.1125)
 		(end 91.6875 107.625)
@@
 		(net 17)
 	)
-	(via
-		(at 91.2 111.55)
-		(size 0.6)
-		(drill 0.3)
-		(layers "F.Cu" "B.Cu")
+	(segment
+		(start 91.2 111.55)
+		(end 91.175 111.575)
+		(width 0.5)
+		(layer "F.Cu")
 		(net 17)
 	)
@@
 		(layer "B.Cu")
 		(net 17)
-	)
-	(segment
-		(start 91.2 114.57)
-		(end 91.2 111.55)
-		(width 0.5)
-		(layer "B.Cu")
-		(net 17)
