File: PS-PowerSelectorPCB.kicad_sch (KiCad schematic)
At the start: 11 parts, among them J1 SuppChargerIn, J2 PowerSupplyIn, J3 Dash_SW, J4 Ext_Power, J5 Src_Select, SW1 Power Source Selector

Commit message: new pinouts
Parts:
- removed J3: Dash_SW, symbol Connector_Generic:Conn_01x03
- removed J5: Src_Select, symbol Connector_Generic:Conn_01x03
- added J3, J5: Conn_01x02, symbol Connector_Generic:Conn_01x02
Connections:
- net LV-: now also J3.1 (Pin_1)
- net LV_EN: now also J3.2 (Pin_2)
- net LV_EN_PS: now also J5.2 (Pin_2)
- net LV_EN_SUPP: now also J5.1 (Pin_1)
Changed lines of the file:
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@@
 	(wire
 		(pts
-			(xy 86.36 62.23) (xy 100.33 62.23)
+			(xy 86.36 57.15) (xy 100.33 57.15)
 		)
 		(stroke
@@
 	(wire
 		(pts
-			(xy 49.53 45.72) (xy 52.07 45.72)
-		)
-		(stroke
-			(width 0)
-			(type default)
-		)
-	)
-	(wire
-		(pts
-			(xy 97.79 57.15) (xy 100.33 57.15)
-		)
-		(stroke
-			(width 0)
-			(type default)
-		)
-	)
-	(wire
-		(pts
-			(xy 86.36 59.69) (xy 100.33 59.69)
+			(xy 86.36 54.61) (xy 100.33 54.61)
 		)
 		(stroke
@@
 	)
 	(label "LV_EN_PS"
-		(at 86.36 62.23 180)
+		(at 86.36 57.15 180)
 		(effects
 			(font
@@
 	)
 	(label "LV_EN_SUPP"
-		(at 86.36 59.69 180)
+		(at 86.36 54.61 180)
 		(effects
 			(font
@@
 	)
 	(symbol
+		(lib_id "Connector_Generic:Conn_01x02")
+		(at 105.41 54.61 0)
+		(unit 1)
+		(exclude_from_sim no)
+		(in_bom yes)
+		(on_board yes)
+		(dnp no)
+		(fields_autoplaced yes)
+		(property "Reference" "J5"
+			(at 107.95 54.6099 0)
+			(effects
+				(font
+					(size 1.27 1.27)
+				)
+				(justify left)
+			)
+		)
+		(property "Value" "Conn_01x02"
+			(at 107.95 57.1499 0)
+			(effects
+				(font
+					(size 1.27 1.27)
+				)
+				(justify left)
+			)
+		)
+		(property "Footprint" ""
+			(at 105.41 54.61 0)
+			(effects
+				(font
+					(size 1.27 1.27)
+				)
+				(hide yes)
+			)
+		)
+		(property "Datasheet" "~"
+			(at 105.41 54.61 0)
+			(effects
+				(font
+					(size 1.27 1.27)
+				)
+				(hide yes)
+			)
+		)
+		(property "Description" "Generic connector, single row, 01x02, script generated (kicad-library-utils/schlib/autogen/connector/)"
+			(at 105.41 54.61 0)
+			(effects
+				(font
+					(size 1.27 1.27)
+				)
+				(hide yes)
+			)
+		)
+		(pin "1"
+		)
+		(pin "2"
+		)
+		(instances
+			(project ""
+				(path "/2c6c62a0-836d-46e8-bf09-ce486c08f53d"
+					(reference "J5")
+					(unit 1)
+				)
+			)
+		)
+	)
+	(symbol
 		(lib_id "power:GND")
 		(at 44.45 36.83 270)
@@
 	)
 	(symbol
-		(lib_id "Connector_Generic:Conn_01x03")
-		(at 57.15 48.26 0)
-		(unit 1)
-		(exclude_from_sim no)
-		(in_bom yes)
-		(on_board yes)
-		(dnp no)
-		(fields_autoplaced yes)
-		(property "Reference" "J3"
-			(at 59.69 46.9899 0)
-			(effects
-				(font
-					(size 1.27 1.27)
-				)
-				(justify left)
-			)
-		)
-		(property "Value" "Dash_SW"
-			(at 59.69 49.5299 0)
-			(effects
-				(font
-					(size 1.27 1.27)
-				)
-				(justify left)
-			)
-		)
-		(property "Footprint" ""
-			(at 57.15 48.26 0)
-			(effects
-				(font
-					(size 1.27 1.27)
-				)
-				(hide yes)
-			)
-		)
-		(property "Datasheet" "~"
-			(at 57.15 48.26 0)
-			(effects
-				(font
-					(size 1.27 1.27)
-				)
-				(hide yes)
-			)
-		)
-		(property "Description" "Generic connector, single row, 01x03, script generated (kicad-library-utils/schlib/autogen/connector/)"
-			(at 57.15 48.26 0)
-			(effects
-				(font
-					(size 1.27 1.27)
-				)
-				(hide yes)
-			)
-		)
-		(pin "3"
-		)
-		(pin "2"
-		)
-		(pin "1"
-		)
-		(instances
-			(project ""
-				(path "/2c6c62a0-836d-46e8-bf09-ce486c08f53d"
-					(reference "J3")
-					(unit 1)
-				)
-			)
-		)
-	)
-	(symbol
 		(lib_id "power:GND")
 		(at 44.45 57.15 270)
@@
 	)
 	(symbol
-		(lib_id "power:+12V")
-		(at 97.79 57.15 90)
-		(unit 1)
-		(exclude_from_sim no)
-		(in_bom yes)
-		(on_board yes)
-		(dnp no)
-		(property "Reference" "#PWR05"
-			(at 101.6 57.15 0)
-			(effects
-				(font
-					(size 1.27 1.27)
-				)
-				(hide yes)
-			)
-		)
-		(property "Value" "LV+"
-			(at 94.488 56.896 90)
+		(lib_id "Connector_Generic:Conn_01x02")
+		(at 57.15 48.26 0)
+		(unit 1)
+		(exclude_from_sim no)
+		(in_bom yes)
+		(on_board yes)
+		(dnp no)
+		(fields_autoplaced yes)
+		(property "Reference" "J3"
+			(at 59.69 48.2599 0)
 			(effects
 				(font
@@
 			)
 		)
-		(property "Footprint" ""
-			(at 97.79 57.15 0)
-			(effects
-				(font
-					(size 1.27 1.27)
-				)
-				(hide yes)
-			)
-		)
-		(property "Datasheet" ""
-			(at 97.79 57.15 0)
-			(effects
-				(font
-					(size 1.27 1.27)
-				)
-				(hide yes)
-			)
-		)
-		(property "Description" "Power symbol creates a global label with name \"+12V\""
-			(at 97.79 57.15 0)
-			(effects
-				(font
-					(size 1.27 1.27)
-				)
-				(hide yes)
-			)
-		)
-		(pin "1"
+		(property "Value" "Conn_01x02"
+			(at 59.69 50.7999 0)
+			(effects
+				(font
+					(size 1.27 1.27)
+				)
+				(justify left)
+			)
+		)
+		(property "Footprint" ""
+			(at 57.15 48.26 0)
+			(effects
+				(font
+					(size 1.27 1.27)
+				)
+				(hide yes)
+			)
+		)
+		(property "Datasheet" "~"
+			(at 57.15 48.26 0)
+			(effects
+				(font
+					(size 1.27 1.27)
+				)
+				(hide yes)
+			)
+		)
+		(property "Description" "Generic connector, single row, 01x02, script generated (kicad-library-utils/schlib/autogen/connector/)"
+			(at 57.15 48.26 0)
+			(effects
+				(font
+					(size 1.27 1.27)
+				)
+				(hide yes)
+			)
+		)
+		(pin "1"
+		)
+		(pin "2"
 		)
 		(instances
 			(project "PS-PowerSelectorPCB"
 				(path "/2c6c62a0-836d-46e8-bf09-ce486c08f53d"
-					(reference "#PWR05")
-					(unit 1)
-				)
-			)
-		)
-	)
-	(symbol
-		(lib_id "power:+12V")
-		(at 49.53 45.72 90)
-		(unit 1)
-		(exclude_from_sim no)
-		(in_bom yes)
-		(on_board yes)
-		(dnp no)
-		(property "Reference" "#PWR07"
-			(at 53.34 45.72 0)
-			(effects
-				(font
-					(size 1.27 1.27)
-				)
-				(hide yes)
-			)
-		)
-		(property "Value" "LV+"
-			(at 46.228 45.466 90)
-			(effects
-				(font
-					(size 1.27 1.27)
-				)
-				(justify left)
-			)
-		)
-		(property "Footprint" ""
-			(at 49.53 45.72 0)
-			(effects
-				(font
-					(size 1.27 1.27)
-				)
-				(hide yes)
-			)
-		)
-		(property "Datasheet" ""
-			(at 49.53 45.72 0)
-			(effects
-				(font
-					(size 1.27 1.27)
-				)
-				(hide yes)
-			)
-		)
-		(property "Description" "Power symbol creates a global label with name \"+12V\""
-			(at 49.53 45.72 0)
-			(effects
-				(font
-					(size 1.27 1.27)
-				)
-				(hide yes)
-			)
-		)
-		(pin "1"
-		)
-		(instances
-			(project "PS-PowerSelectorPCB"
-				(path "/2c6c62a0-836d-46e8-bf09-ce486c08f53d"
-					(reference "#PWR07")
+					(reference "J3")
 					(unit 1)
 				)
@@
 					(unit 1)
 				)
-			)
-		)
-	)
-	(symbol
-		(lib_id "Connector_Generic:Conn_01x03")
-		(at 105.41 59.69 0)
-		(unit 1)
-		(exclude_from_sim no)
-		(in_bom yes)
-		(on_board yes)
-		(dnp no)
-		(fields_autoplaced yes)
-		(property "Reference" "J5"
-			(at 107.95 58.4199 0)
-			(effects
-				(font
-					(size 1.27 1.27)
-				)
-				(justify left)
-			)
-		)
-		(property "Value" "Src_Select"
-			(at 107.95 60.9599 0)
-			(effects
-				(font
-					(size 1.27 1.27)
-				)
-				(justify left)
-			)
-		)
-		(property "Footprint" ""
-			(at 105.41 59.69 0)
-			(effects
-				(font
-					(size 1.27 1.27)
-				)
-				(hide yes)
-			)
-		)
-		(property "Datasheet" "~"
-			(at 105.41 59.69 0)
-			(effects
-				(font
-					(size 1.27 1.27)
-				)
-				(hide yes)
-			)
-		)
-		(property "Description" "Generic connector, single row, 01x03, script generated (kicad-library-utils/schlib/autogen/connector/)"
-			(at 105.41 59.69 0)
-			(effects
-				(font
-					(size 1.27 1.27)
-				)
-				(hide yes)
-			)
-		)
-		(pin "3"
-		)
-		(pin "2"
-		)
-		(pin "1"
-		)
-		(instances
-			(project "PS-PowerSelectorPCB"
-				(path "/2c6c62a0-836d-46e8-bf09-ce486c08f53d"
-					(reference "J5")
-					(unit 1)
-				)

Commit message: initial schematic
Parts:
- removed J4: Ext_Power, symbol Connector_Generic:Conn_01x03
- removed J5: Conn_01x02, symbol Connector_Generic:Conn_01x02
- added D6, D7: D_Schottky, symbol Device:D_Schottky
- added F1: 5A, footprints:FUSE_3568, symbol 3568:3568
- added F2: 100mA, symbol Device:Polyfuse
- added H1, H2, H3, H4: MountingHole, MountingHole:MountingHole_3.2mm_M3, symbol Mechanical:MountingHole
- added J4: PowerSupplyOut, UTSVT_Connectors:AMASS_XT30PW-M_1x02_P2.50mm_Horizontal, symbol Connector_Generic:Conn_01x02
- added J5: Signals, Connector_Molex:Molex_Nano-Fit_105309-xx06_1x06_P2.50mm_Vertical, symbol Connector_Generic:Conn_01x06
- added J6: HV_Lockout, UTSVT_Connectors:Molex_Nano-Fit_105309-xx02_1x02_P2.50mm_Vertical, symbol Connector_Generic:Conn_01x02
- added LOGO1: LHRS, UTSVT_Logos:LHRs_LOGO, symbol utsvt_misc:Logo_Placeholder
- added LOGO2: Hallock, UTSVT_Logos:Hallock_Image_Tiny, symbol utsvt_misc:Logo_Placeholder
- added R1, R2, R3, R4, R5: 1k, symbol Device:R_US
- D2: value PowerSupplyIn -> PS_In
- D4: value PowerSupplySelected -> PS_Sel
- D5: value SuppSelected' -> Supp_Sel
- J1: footprint (none) -> Connector_AMASS:AMASS_XT60-M_1x02_P7.20mm_Vertical
- J2: footprint (none) -> UTSVT_Connectors:AMASS_XT30PW-M_1x02_P2.50mm_Horizontal
- J3: value Conn_01x02 -> SuppChargerOut; footprint (none) -> Connector_AMASS:AMASS_XT60-M_1x02_P7.20mm_Vertical
Connections:
- net LV-: now also J4.1 (Pin_1), J5.1 (Pin_1), R1.2, R2.2
- net LV_EN_PS: now also J5.6 (Pin_6), R4.2
- net LV_EN_SUPP: now also J5.5 (Pin_5), R5.2
- net PS+: now also D2.2 (A), D6.2 (A), J4.2 (Pin_2)
- net SuppChargerIn+: now also D1.2 (A), F1.1, F1.3; no longer SW1.5 (B)
- net SuppChargerOut+: now also J3.2 (Pin_2)
- net at D5.1 (K): now also R5.1
- net LED+: now reaches D5.2 (A)
- net LED+: now also D3.2 (A), D4.2 (A), D6.1 (K), D7.1 (K)
- net at D2.1 (K): now also R2.1
- net at D4.1 (K): now also R4.1
- net at D3.1 (K): now also R3.1
- net at D1.1 (K): now also R1.1
- net LV_EN renamed LV_EN_FUSED
- net LV_EN_FUSED: now also F2.2, R3.2; no longer J3.2 (Pin_2)
- new net HV_LO+: J5.3 (Pin_3), J6.1 (Pin_1)
- new net HV_LO-: J5.4 (Pin_4), J6.2 (Pin_2)
- new net LV_EN_IN: F2.1, J5.2 (Pin_2)
- new net SC_Fused: D7.2 (A), F1.2, F1.4
- new net SuppChargerFused: SW1.5 (B)
Other:
- note added: "Blue LEDs: Inom = 20mA, Imax = 80mA, Vf = 2.7-3.1V SuppCharger: 18-32V (24V nom) LED current draw: 15-29mA (20mA nom)"
- note added: "From Dash"
- note added: "Red LEDs: Inom = 25mA, Imax = 50mA, Vf = 1.6-2.6V SuppCharger: 18-32V (24V nom) LED current draw: 15-30mA (22mA nom)"
- note added: "To PDE"
- note added: "check this ptc fuse"
- note removed: "Regulate supp charger power for charging led (assume 18-32V input)"
- moved on the sheet: D1, D2, D3, D4, D5, SW1A, SW1B

Commit message: initial layout
Parts:
- added S1: 100DP1T2B4VS2QE, footprints:100DP1T2B4VS2QE, symbol 100DP1T2B4VS2QE:100DP1T2B4VS2QE
- D1, D2, D3, D4, D5: footprint (none) -> LED_SMD:LED_0603_1608Metric_Pad1.05x0.95mm_HandSolder
- D6, D7: footprint (none) -> Diode_SMD:D_SOD-123
- F2: footprint (none) -> Fuse:Fuse_1210_3225Metric_Pad1.42x2.65mm_HandSolder
- J2, J4: footprint UTSVT_Connectors:AMASS_XT30PW-M_1x02_P2.50mm_Horizontal -> footprints:AMASS_XT30UPB-M_1x02_P5.0mm_Vertical
- R1, R2, R3, R4, R5: footprint (none) -> Resistor_SMD:R_0603_1608Metric_Pad0.98x0.95mm_HandSolder
- SW1: footprint (none) -> footprints:100DP1T2B4VS2QE; P/N (none) -> 612-100DP1T2B4VS2QE; now not fitted
Connections:
- net SuppChargerFused is gone; now on net SC_Fused: SW1.5 (B)
- net LV_EN_FUSED: now also S1.2 (COM1)
- net LV_EN_PS: now also S1.3 (NO1)
- net LV_EN_SUPP: now also S1.1 (NC1)
- net SC_Fused: now also S1.5 (COM2)
- net SuppChargerOut+: now also S1.6 (NO2)
- no-connect marks 1 -> 6
Other:
- moved on the sheet: D1, D2, D3, D4, D5, D6, D7, F1, F2, H1, H2, H3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

Commit message: fixed switch footprint + silkscreen
Parts:
- removed S1: 100DP1T2B4VS2QE, footprints:100DP1T2B4VS2QE, symbol 100DP1T2B4VS2QE:100DP1T2B4VS2QE
- SW1: now fitted
Connections:
- no-connect marks 6 -> 1

Commit message: bomb
Parts:
- D1, D2: P/N (none) -> XL-1608UBC-06A
- D3, D4, D5: P/N (none) -> NCD0603R1
- D6, D7: P/N (none) -> 1N5819HW-7-F
- F1: MANUFACTURER Keystone -> (none); MAXIMUM_PACKAGE_HEIGHT 7.37 mm -> (none); P/N (none) -> 3568; PARTREV C -> (none); SNAPEDA_PN 3568 -> (none); STANDARD Manufacturer Recommendations -> (none)
- F2: P/N (none) -> SMD1210B005TF
- J1, J3: P/N (none) -> XT60-M
- J2, J4: P/N (none) -> XT30UPB-M
- J5: P/N (none) -> 1053091206
- J6: P/N (none) -> 1053091202
- R1, R2, R3, R4, R5: P/N (none) -> CRCW06031K00FKEI
Other:
- note removed: "check this ptc fuse"
Changed lines of the file:
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@@
 		)
 	)
-	(text "check this ptc fuse"
-		(exclude_from_sim no)
-		(at 115.824 92.202 0)
-		(effects
-			(font
-				(size 1.27 1.27)
-			)
-		)
-	)
 	(text "XT60\n"
 		(exclude_from_sim no)
@@
 			)
 		)
+		(property "P/N" "CRCW06031K00FKEI"
+			(at 116.84 156.21 0)
+			(effects
+				(font
+					(size 1.27 1.27)
+				)
+				(hide yes)
+			)
+		)
 		(pin "1"
 		)
@@
 			)
 		)
-		(property "Description" "Red LED, P/N: NCD0603R1"
+		(property "Description" "Red LED"
 			(at 116.84 146.05 0)
 			(effects
@@
 			)
 		)
-		(property "Sim.Pins" "1=K 2=A"
+		(property "P/N" "NCD0603R1"
 			(at 116.84 146.05 0)
 			(effects
@@
 			)
 		)
+		(property "P/N" "1053091206"
+			(at 69.85 73.66 0)
+			(effects
+				(font
+					(size 1.27 1.27)
+				)
+				(hide yes)
+			)
+		)
 		(pin "2"
 		)
@@
 			)
 		)
-		(property "Description" "MF-USHT010KX/36-2"
+		(property "Description" "PTC fuse"
 			(at 114.3 88.9 0)
 			(effects
@@
 			)
 		)
+		(property "P/N" "SMD1210B005TF"
+			(at 114.3 88.9 90)
+			(effects
+				(font
+					(size 1.27 1.27)
+				)
+				(hide yes)
+			)
+		)
 		(pin "1"
 		)
@@
 			)
 		)
-		(property "Description" "Blue LED, P/N: XL-1608UBC-06A"
+		(property "Description" "Blue LED"
 			(at 48.26 146.05 0)
 			(effects
@@
 			)
 		)
-		(property "Sim.Pins" "1=K 2=A"
+		(property "P/N" "XL-1608UBC-06A"
 			(at 48.26 146.05 0)
 			(effects
@@
 			)
 		)
+		(property "P/N" "CRCW06031K00FKEI"
+			(at 97.79 156.21 0)
+			(effects
+				(font
+					(size 1.27 1.27)
+				)
+				(hide yes)
+			)
+		)
 		(pin "1"
 		)
@@
 			)
 		)
-		(property "Description" ""
-			(at 114.3 74.93 0)
-			(effects
-				(font
-					(size 1.27 1.27)
-				)
-				(hide yes)
-			)
-		)
-		(property "PARTREV" "C"
-			(at 114.3 74.93 0)
-			(effects
-				(font
-					(size 1.27 1.27)
-				)
-				(justify bottom)
-				(hide yes)
-			)
-		)
-		(property "MANUFACTURER" "Keystone"
+		(property "Description" "SMD fuse holder"
 			(at 114.3 74.93 0)
 			(effects
@@
 					(size 1.27 1.27)
 				)
-				(justify bottom)
 				(hide yes)
 			)
 		)
-		(property "SNAPEDA_PN" "3568"
-			(at 114.3 74.93 0)
-			(effects
-				(font
-					(size 1.27 1.27)
-				)
-				(justify bottom)
-				(hide yes)
-			)
-		)
-		(property "MAXIMUM_PACKAGE_HEIGHT" "7.37 mm"
-			(at 114.3 74.93 0)
-			(effects
-				(font
-					(size 1.27 1.27)
-				)
-				(justify bottom)
-				(hide yes)
-			)
-		)
-		(property "STANDARD" "Manufacturer Recommendations"
+		(property "P/N" "3568"
 			(at 114.3 74.93 0)
 			(effects
@@
 			)
 		)
-		(property "Description" "1N5819HW-7-F"
+		(property "Description" ""
 			(at 143.51 154.94 0)
 			(effects
@@
 			)
 		)
+		(property "P/N" "1N5819HW-7-F"
+			(at 143.51 154.94 90)
+			(effects
+				(font
+					(size 1.27 1.27)
+				)
+				(hide yes)
+			)
+		)
 		(pin "1"
 		)
@@
 			)
 		)
+		(property "P/N" "XT30UPB-M"
+			(at 53.34 41.91 0)
+			(effects
+				(font
+					(size 1.27 1.27)
+				)
+				(hide yes)
+			)
+		)
 		(pin "1"
 		)
@@
 			)
 		)
+		(property "P/N" "CRCW06031K00FKEI"
+			(at 48.26 156.21 0)
+			(effects
+				(font
+					(size 1.27 1.27)
+				)
+				(hide yes)
+			)
+		)
 		(pin "1"
 		)
@@
 			)
 		)
+		(property "P/N" "XT30UPB-M"
+			(at 118.11 43.18 0)
+			(effects
+				(font
+					(size 1.27 1.27)
+				)
+				(hide yes)
+			)
+		)
 		(pin "1"
 		)
@@
 			)
 		)
-		(property "Description" "Red LED, P/N: NCD0603R1"
+		(property "Description" "Red LED"
 			(at 97.79 146.05 0)
 			(effects
@@
 			)
 		)
-		(property "Sim.Pins" "1=K 2=A"
+		(property "P/N" "NCD0603R1"
 			(at 97.79 146.05 0)
 			(effects
@@
 			)
 		)
+		(property "P/N" "XT60-M"
+			(at 118.11 27.94 0)
+			(effects
+				(font
+					(size 1.27 1.27)
+				)
+				(hide yes)
+			)
+		)
 		(pin "2"
 		)
@@
 			)
 		)
+		(property "P/N" "CRCW06031K00FKEI"
+			(at 29.21 156.21 0)
+			(effects
+				(font
+					(size 1.27 1.27)
+				)
+				(hide yes)
+			)
+		)
 		(pin "1"
 		)
@@
 			)
 		)
-		(property "Description" "Red LED, P/N: NCD0603R1"
+		(property "Description" "Red LED"
 			(at 78.74 146.05 0)
 			(effects
@@
 			)
 		)
-		(property "Sim.Pins" "1=K 2=A"
+		(property "P/N" "NCD0603R1"
 			(at 78.74 146.05 0)
 			(effects
@@
 			)
 		)
-		(property "Description" "Blue LED, P/N: XL-1608UBC-06A"
+		(property "Description" "Blue LED"
 			(at 29.21 146.05 0)
 			(effects
@@
 			)
 		)
-		(property "Sim.Pins" "1=K 2=A"
-			(at 29.21 146.05 0)
+		(property "P/N" "XL-1608UBC-06A"
+			(at 29.21 146.05 90)
 			(effects
 				(font
@@
 			)
 		)
+		(property "P/N" "XT60-M"
+			(at 53.34 27.94 0)
+			(effects
+				(font
+					(size 1.27 1.27)
+				)
+				(hide yes)
+			)
+		)
 		(pin "2"
 		)
@@
 			)
 		)
+		(property "P/N" "1053091202"
+			(at 69.85 86.36 0)
+			(effects
+				(font
+					(size 1.27 1.27)
+				)
+				(hide yes)
+			)
+		)
 		(pin "1"
 		)
@@
 			)
 		)
+		(property "P/N" "CRCW06031K00FKEI"
+			(at 78.74 156.21 0)
+			(effects
+				(font
+					(size 1.27 1.27)
+				)
+				(hide yes)
+			)
+		)
 		(pin "1"
 		)
@@
 			)
 		)
-		(property "Description" "1N5819HW-7-F"
+		(property "Description" ""
 			(at 148.59 154.94 0)
 			(effects
 				(font
+					(size 1.27 1.27)
+				)
+				(hide yes)
+			)
+		)
+		(property "P/N" "1N5819HW-7-F"
+			(at 148.59 154.94 90)
+			(effects
+				(font
